File: ZXCT1008_over.kicad_sch (KiCad schematic)
At the start: 15 parts, among them Q1 FMMT597, U1 SMAZ15, U2 ZXCT1008F, U3 C1608C0G2A100D080AA_p, U4 DI_BZX84C4V7, U5 C2012C0G2A102J060AA_p

Commit message: simulation
load regulation simulation
Parts:
- I1: value IDC -> {ILOAD}; symbol Simulation_SPICE:IDC -> ZXCT1008F:IDC; Spice_Model {ILOAD} -> (none); Spice_Netlist_Enabled Y -> (none); Spice_Primitive I -> (none)
- Q1: symbol Device:Q_PNP_CBE -> ZXCT1008F:Q_PNP_CBE; Spice_Lib_File models/FMMT597.spice.txt -> (none); Spice_Model FMMT597 -> (none); Spice_Netlist_Enabled Y -> (none); Spice_Primitive Q -> (none)
- R1: symbol Device:R -> ZXCT1008F:R_3
- R2: symbol Device:R -> ZXCT1008F:R_6
- R3: symbol Device:R -> ZXCT1008F:R_2
- R4: symbol Device:R -> ZXCT1008F:R_1
- R5: symbol Device:R -> ZXCT1008F:R_5
- R6: symbol Device:R -> ZXCT1008F:R_4
- R7: symbol Device:R -> ZXCT1008F:R
- U1: symbol Simulation_SPICE:DIODE -> ZXCT1008F:DIODE; Spice_Lib_File models/SMAZ15.spice.txt -> (none); Spice_Model SMAZ15 -> (none); Spice_Netlist_Enabled Y -> (none); Spice_Primitive X -> (none)
- U2: Spice_Lib_File models/ZXCT1008F.spice.txt -> (none); Spice_Model ZXCT1008F -> (none); Spice_Netlist_Enabled Y -> (none); Spice_Primitive X -> (none)
- U3: symbol Device:C -> ZXCT1008F:C; Spice_Lib_File models/C1608C0G2A100D080AA_p.mod -> (none); Spice_Model C1608C0G2A100D080AA_p -> (none); Spice_Netlist_Enabled Y -> (none); Spice_Primitive X -> (none)
- U4: symbol Simulation_SPICE:DIODE -> ZXCT1008F:DIODE_1; Spice_Lib_File models/BZX84C4V7.spice.txt -> (none); Spice_Model DI_BZX84C4V7 -> (none); Spice_Netlist_Enabled Y -> (none); Spice_Primitive X -> (none)
- U5: symbol Device:C -> ZXCT1008F:C_1; Spice_Lib_File models/C2012C0G2A102J060AA_p.mod -> (none); Spice_Model C2012C0G2A102J060AA_p -> (none); Spice_Netlist_Enabled Y -> (none); Spice_Primitive X -> (none)
- V1: value VDC -> {VSOURCE}; symbol Simulation_SPICE:VDC -> ZXCT1008F:VDC; Spice_Model {VSOURCE} -> (none); Spice_Netlist_Enabled Y -> (none); Spice_Primitive V -> (none)
